File: C64ExpansionBreakout.sch (KiCad schematic (older format))
At the start: 5 parts, among them J1 Power, J2 GND, J3 Breakout, SW1 Reset, U1 C64-Exp-Port

Commit message: Copied/rescued connector symbols.
Parts:
- J1: symbol Connector:Conn_02x02_Odd_Even -> C64-Exp-Port:Conn_02x02_Odd_Even
- J2: symbol Connector:Conn_01x02 -> C64-Exp-Port:Conn_01x02
Changed lines of the file:
@@
 EESchema Schematic File Version 4
+LIBS:C64ExpansionBreakout-cache
 EELAYER 26 0
 EELAYER END
@@
 GND
 $Comp
-L Connector:Conn_02x02_Odd_Even J1
+L C64-Exp-Port:Conn_02x02_Odd_Even J1
 U 1 1 5ACD4D51
 P 1400 1100
@@
 A0
 $Comp
-L Connector:Conn_01x02 J2
+L C64-Exp-Port:Conn_01x02 J2
 U 1 1 5ACD5626
 P 1450 1600
