File: C64ExpansionBreakout.sch (KiCad schematic (older format))
At the start: 5 parts, among them J1 Power, J2 GND, J3 Breakout, SW1 Reset, U1 C64-Exp-Port

Commit message: Added 27C512 / 27C020 Eprom socket.
Parts:
- added J4: Other, Socket_Strips:Socket_Strip_Straight_1x06_Pitch2.54mm, symbol Connector:Conn_01x06_Female
- added J5: Config, Pin_Headers:Pin_Header_Straight_2x02_Pitch2.54mm, symbol C64-Exp-Port:Conn_02x02_Odd_Even
- added JP1: 27c512, Pin_Headers:Pin_Header_Straight_1x02_Pitch2.54mm, symbol device:Jumper_NO_Small
- added U2: 27C512, Housings_DIP:DIP-32_W15.24mm_Socket_LongPads, symbol memory:27C020
Connections:
- net labels added: +5V, CE, OA13, OA14, OA15, OA16, OA17
- net labels removed: 5V
- wire segments 0 -> 34

Commit message: Finalizing revision 2.
Parts:
- added C1: 100n, Capacitors_THT:C_Disc_D4.3mm_W1.9mm_P5.00mm, symbol device:C
Changed lines of the file:
@@
 Sheet 1 1
 Title "C64ExpansionBreakout"
-Date ""
-Rev ""
+Date "2018-09-07"
+Rev "Rev.2"
 Comp "hackup.net"
 Comment1 ""
@@
 Connection ~ 2400 6050
 Connection ~ 1850 5950
+$Comp
+L device:C C1
+U 1 1 5B921DF0
+P 3700 5850
+F 0 "C1" H 3815 5896 50  0000 L CNN
+F 1 "100n" H 3815 5805 50  0000 L CNN
+F 2 "Capacitors_THT:C_Disc_D4.3mm_W1.9mm_P5.00mm" H 3738 5700 50  0001 C CNN
+F 3 "~" H 3700 5850 50  0001 C CNN
+	1    3700 5850
+	1    0    0    -1
+$EndComp
+$Comp
+L power:+5V #PWR0111
+U 1 1 5B921ECA
+P 3700 5700
+F 0 "#PWR0111" H 3700 5550 50  0001 C CNN
+F 1 "+5V" H 3715 5873 50  0000 C CNN
+F 2 "" H 3700 5700 50  0001 C CNN
+F 3 "" H 3700 5700 50  0001 C CNN
+	1    3700 5700
+	1    0    0    -1
+$EndComp
+$Comp
+L power:GND #PWR0112
+U 1 1 5B921EE9
+P 3700 6000
+F 0 "#PWR0112" H 3700 5750 50  0001 C CNN
+F 1 "GND" H 3705 5827 50  0000 C CNN
+F 2 "" H 3700 6000 50  0001 C CNN
+F 3 "" H 3700 6000 50  0001 C CNN
+	1    3700 6000
+	1    0    0    -1
+$EndComp
 $EndSCHEMATC

Commit message: Clean up libs.
Parts:
- U1: footprint Sukko:C64-Cart-NoSilkS -> C64-Exp-Port:C64-Cart-NoSilkS
Changed lines of the file:
@@
 Sheet 1 1
 Title "C64ExpansionBreakout"
-Date "2018-09-07"
-Rev "Rev.2"
+Date "2018-10-07"
+Rev "Rev. 2.1"
 Comp "hackup.net"
 Comment1 ""
@@
 F 0 "U1" H 7550 4415 50  0000 C CNN
 F 1 "C64-Exp-Port" H 7550 4324 50  0000 C CNN
-F 2 "Sukko:C64-Cart-NoSilkS" H 7550 1550 50  0001 C CNN
+F 2 "C64-Exp-Port:C64-Cart-NoSilkS" H 7550 1550 50  0001 C CNN
 F 3 "DOCUMENTATION" H 7550 1450 50  0001 C CNN
 	1    7550 3000
