File: C64ExpansionBreakout.kicad_pcb (KiCad board)
At the start: 2 copper layers, 99.1 x 82.4 mm, 11 parts, among them J1 Power, J2 GND, J3 Breakout, J4 Other, J5 Config, SW1 Reset, U1 C64-Exp-Port, U2 27C512

Commit message: Revision update.
Other:
- board text added: "Rev. 2.1 github.com/hackup/C64ExpansionBreakout"
- board text removed: "Rev.2 github.com/hackup/C64ExpansionBreakout"
Changed lines of the file:
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@@
     (title C64ExpansionBreakout)
     (date 2018-09-07)
-    (rev Rev.2)
+    (rev "Rev. 2.1")
     (company hackup.net)
   )
@@
   (gr_line (start 100.203 104.648) (end 98.552 103.124) (angle 90) (layer Edge.Cuts) (width 0.15))
   (gr_line (start 100.203 140.716) (end 100.203 104.648) (angle 90) (layer Edge.Cuts) (width 0.15))
-  (gr_text "Rev.2\ngithub.com/hackup/C64ExpansionBreakout" (at 196.85 102.108) (layer F.SilkS)
+  (gr_text "Rev. 2.1\ngithub.com/hackup/C64ExpansionBreakout" (at 196.85 102.108) (layer F.SilkS)
     (effects (font (size 1.5 1.5) (thickness 0.3)) (justify right))
   )
