File: C64ExpansionBreakout.kicad_pcb (KiCad board)
At the start: 2 copper layers, 99.1 x 82.4 mm, 11 parts, among them J1 Power, J2 GND, J3 Breakout, J4 Other, J5 Config, SW1 Reset, U1 C64-Exp-Port, U2 27C512

Commit message: Clean up libs.
Parts:
- U1: footprint Sukko:C64-Cart-NoSilkS -> C64-Exp-Port:C64-Cart-NoSilkS
